Commit message: changed mesh path in urdf

File: velodyne_description/urdf/VLP-16.urdf.xacro (robot description, xacro)
@@ -16,10 +16,10 @@
       <visual>
         <geometry>
-          <mesh filename="package://velodyne_description/meshes/VLP16_base_1.dae"/>
+          <mesh filename="file://$(find velodyne_description)/meshes/VLP16_base_1.dae"/>
         </geometry>
       </visual>
       <visual>
         <geometry>
-          <mesh filename="package://velodyne_description/meshes/VLP16_base_2.dae"/>
+          <mesh filename="file://$(find velodyne_description)/meshes/VLP16_base_2.dae"/>
         </geometry>
       </visual>

Commit message: fixup

File: velodyne_description/urdf/VLP-16.urdf.xacro (robot description, xacro)
@@ -45,5 +45,5 @@
         <origin xyz="0 0 -0.0377"/>
         <geometry>
-          <mesh filename="package://velodyne_description/meshes/VLP16_scan.dae"/>
+          <mesh filename="file://$(find velodyne_description)/meshes/VLP16_scan.dae"/>
         </geometry>
       </visual>
@@ -129,4 +129,5 @@
             <min_range>${min_range}</min_range>
             <max_range>${max_range}</max_range>
+            <min_intensity>0.0</min_intensity>
             <gaussianNoise>${noise}</gaussianNoise>
           </plugin>
